File: MQTT-Module-CurrentSensors.kicad_pcb (KiCad board)
At the start: 4 copper layers, 44 x 58.4 mm, 66 parts, among them IC401 16 Bit ADC, J301 A2541WV-10P, J302 A2541WV-10P, J303 A2541WV-2x3P, J304 1715747, U201 ATmega328PB-A, U501 Precision ZD RR, U502 Precision ZD RR, U503 Precision ZD RR

Commit message: Update
Parts:
- added G***: LOGO, LOGO, F.Cu at (156.9, 133.2)
- added G***: LOGO, LOGO, B.Cu at (140.1, 111.8)
- moved R505 2.09 mm to (128.0, 108.7), turned to 0 degrees
- moved TP601 0.40 mm to (125.4, 105.9)
Routing:
- net +25V: track 98.8 -> 103.4 mm
- net /AnalogDigitalConverter/Sens2: track 10.5 -> 11.9 mm, vias 0 -> 2
- net /AnalogDigitalConverter/Sens1: track 24.8 -> 24.4 mm, vias 0 -> 2
- net GND: vias 60 -> 63
Other:
- board text added: "github.com/WiddleWabbit/ MQTT-Module-Sensor"

Commit message: Added License to Board
Parts:
- moved G*** 3.13 mm to (140.5, 108.7)
Other:
- board text added: "Licensed under CERN-OHL-P v2"
Changed lines of the file:
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@@
 	(footprint "LOGO"
 		(layer "B.Cu")
-		(at 140.1 111.8 180)
+		(at 140.5 108.7 180)
 		(property "Reference" "G***"
 			(at 0 0 0)
@@
 		)
 	)
+	(gr_text "Licensed under CERN-OHL-P v2"
+		(at 140.4 122.1 0)
+		(layer "B.SilkS")
+		(effects
+			(font
+				(size 1.2 1.2)
+				(thickness 0.3)
+				(bold yes)
+			)
+			(justify bottom mirror)
+		)
+	)
 	(gr_text "SNS"
 		(at 155.928572 92.3 -0)
@@
 	)
 	(gr_text "github.com/WiddleWabbit/\nMQTT-Module-Sensor"
-		(at 140 121.1 0)
-		(layer "B.SilkS")
-		(effects
-			(font
-				(size 1.3 1.3)
+		(at 140.5 118.2 0)
+		(layer "B.SilkS")
+		(effects
+			(font
+				(size 1.5 1.5)
 				(thickness 0.325)
 				(bold yes)
