File: adc.kicad_sch (KiCad schematic)
At the start: 4 parts, among them IC401 16 Bit ADC

Commit message: Interactive BOM added. Updated Mega Symbol. Updated symbols in schematic. Generated production files.
Parts:
- R401, R417: Manufacturer (none) -> UNI-ROYAL(Uniroyal Elec); Manufacturer Part No (none) -> 0805W8F4701T5E
Changed lines of the file:
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@@
+			)
+		)
+		(property "Manufacturer" "UNI-ROYAL(Uniroyal Elec)"
+			(at 207.01 776.2 0)
+			(effects
+				(font
+					(size 1.27 1.27)
+				)
+				(justify left top)
+				(hide yes)
+			)
+		)
+		(property "Manufacturer Part No" "0805W8F4701T5E"
+			(at 207.01 876.2 0)
+			(effects
+				(font
+					(size 1.27 1.27)
+				)
+				(justify left top)
+				(hide yes)
 			)
 		)
@@
 				(hide yes)
 			)
+		)
+		(property "Manufacturer" "UNI-ROYAL(Uniroyal Elec)"
+			(at 207.01 795.25 0)
+			(effects
+				(font
+					(size 1.27 1.27)
+				)
+				(justify left top)
+				(hide yes)
+			)
+		)
+		(property "Manufacturer Part No" "0805W8F4701T5E"
+			(at 207.01 895.25 0)
+			(effects
+				(font
+					(size 1.27 1.27)
+				)
+				(justify left top)
+				(hide yes)
+			)
