File: controller.kicad_sch (KiCad schematic)
At the start: 6 parts, among them U201 ATmega328PB-A

Commit message: Interactive BOM added. Updated Mega Symbol. Updated symbols in schematic. Generated production files.
Parts:
- removed U201: ATmega328PB-A, Package_QFP:TQFP-32_7x7mm_P0.8mm, symbol MCU_Microchip_ATmega:ATmega328PB-A
- added U202: ATmega328PB-A, Package_QFP:TQFP-32_7x7mm_P0.8mm, symbol MICROCHIPTECH Microcontrollers:ATmega328PB-A
Connections:
- net +3V3: now also U202.18 (AVCC), U202.4 (VCC)
- net AREF: now also U202.20 (AREF)
- net GND: now also U202.21 (GND), U202.5 (GND)
- net MISO: now also U202.16 (PB4)
- net MOD: now also U202.1 (PD3)
- net MOSI: now also U202.15 (PB3)
- net RESET: now also U202.29 (~{RESET}/PC6)
- net SCK: now also U202.17 (PB5)
- net SCL0: now also U202.3 (PE0)
- net SCL1: now also U202.28 (PC5)
- net SDA0: now also U202.6 (PE1)
- net SDA1: now also U202.27 (PC4)
- net SNS: now also U202.2 (PD4)
Changed lines of the file:
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@@
+	)
+	(symbol
+		(lib_id "MICROCHIPTECH Microcontrollers:ATmega328PB-A")
+		(at 93.98 86.36 0)
+		(unit 1)
+		(exclude_from_sim no)
+		(in_bom yes)
+		(on_board yes)
+		(dnp no)
+		(fields_autoplaced yes)
+		(property "Reference" "U202"
+			(at 96.1233 124.46 0)
+			(effects
+				(font
+					(size 1.27 1.27)
+				)
+				(justify left)
+			)
+		)
+		(property "Value" "ATmega328PB-A"
+			(at 96.1233 127 0)
+			(effects
+				(font
+					(size 1.27 1.27)
+				)
+				(justify left)
+			)
+		)
+		(property "Footprint" "Package_QFP:TQFP-32_7x7mm_P0.8mm"
+			(at 93.98 86.36 0)
+			(effects
+				(font
+					(size 1.27 1.27)
+					(italic yes)
+				)
+				(hide yes)
+			)
+		)
+		(property "Datasheet" "http://ww1.microchip.com/downloads/en/DeviceDoc/40001906C.pdf"
+			(at 93.98 86.36 0)
+			(effects
+				(font
+					(size 1.27 1.27)
+				)
+				(hide yes)
+			)
+		)
+		(property "Description" "20MHz, 32kB Flash, 2kB SRAM, 1kB EEPROM, TQFP-32"
+			(at 93.98 86.36 0)
+			(effects
+				(font
+					(size 1.27 1.27)
+				)
+				(hide yes)
+			)
+		)
+		(property "Manufacturer" "Microchip Tech"
+			(at 93.98 86.36 0)
+			(effects
+				(font
+					(size 1.27 1.27)
+				)
+				(hide yes)
+			)
+		)
+		(property "Manufacturer Part No" "ATMEGA328PB-AU"
+			(at 93.98 86.36 0)
+			(effects
+				(font
+					(size 1.27 1.27)
+				)
+				(hide yes)
+			)
+		)
+		(property "JLCPCB Part #" "C132230"
+			(at 93.98 86.36 0)
+			(effects
+				(font
+					(size 1.27 1.27)
+				)
+				(hide yes)
+			)
+		)
+		(property "Package" "TQFP-32(7x7)"
+			(at 93.98 86.36 0)
+			(effects
+				(font
+					(size 1.27 1.27)
+				)
+				(hide yes)
+			)
+		)
+		(property "Part Type" "Extended"
+			(at 93.98 86.36 0)
+			(effects
+				(font
+					(size 1.27 1.27)
+				)
+				(hide yes)
+			)
+		)
+		(pin "3"
+		)
+		(pin "20"
+		)
+		(pin "22"
+		)
+		(pin "6"
+		)
+		(pin "12"
+		)
+		(pin "14"
+		)
+		(pin "15"
+		)
+		(pin "19"
+		)
+		(pin "4"
+		)
+		(pin "21"
+		)
+		(pin "5"
+		)
+		(pin "18"
+		)
+		(pin "13"
+		)
+		(pin "29"
+		)
+		(pin "31"
+		)
+		(pin "9"
+		)
+		(pin "30"
+		)
+		(pin "23"
+		)
+		(pin "24"
+		)
+		(pin "27"
+		)
+		(pin "28"
+		)
+		(pin "1"
+		)
+		(pin "17"
+		)
+		(pin "25"
+		)
+		(pin "32"
+		)
+		(pin "26"
+		)
+		(pin "11"
+		)
+		(pin "7"
+		)
+		(pin "16"
+		)
+		(pin "8"
+		)
+		(pin "2"
+		)
+		(pin "10"
+		)
+		(instances
+			(project ""
+				(path "/fcdc4d99-6273-4901-9910-bd8fd00b962f/aa87b2dd-90b3-41b3-8e99-8dcc5f11db59"
+					(reference "U202")
+					(unit 1)
+				)
+			)
+		)
 	)
 	(symbol
@@
 					(unit 1)
 				)
-			)
-		)
-	)
-	(symbol
-		(lib_id "MCU_Microchip_ATmega:ATmega328PB-A")
-		(at 93.98 86.36 0)
-		(unit 1)
-		(exclude_from_sim no)
-		(in_bom yes)
-		(on_board yes)
-		(dnp no)
-		(fields_autoplaced yes)
-		(property "Reference" "U201"
-			(at 96.1233 124.46 0)
-			(effects
-				(font
-					(size 1.27 1.27)
-				)
-				(justify left)
-			)
-		)
-		(property "Value" "ATmega328PB-A"
-			(at 96.1233 127 0)
-			(effects
-				(font
-					(size 1.27 1.27)
-				)
-				(justify left)
-			)
-		)
-		(property "Footprint" "Package_QFP:TQFP-32_7x7mm_P0.8mm"
-			(at 93.98 86.36 0)
-			(effects
-				(font
-					(size 1.27 1.27)
-					(italic yes)
-				)
-				(hide yes)
-			)
-		)
-		(property "Datasheet" "http://ww1.microchip.com/downloads/en/DeviceDoc/40001906C.pdf"
-			(at 93.98 86.36 0)
-			(effects
-				(font
-					(size 1.27 1.27)
-				)
-				(hide yes)
-			)
-		)
-		(property "Description" "20MHz, 32kB Flash, 2kB SRAM, 1kB EEPROM, TQFP-32"
-			(at 93.98 86.36 0)
-			(effects
-				(font
-					(size 1.27 1.27)
-				)
-				(hide yes)
-			)
-		)
-		(pin "22"
-		)
-		(pin "20"
-		)
-		(pin "19"
-		)
-		(pin "16"
-		)
-		(pin "3"
-		)
-		(pin "21"
-		)
-		(pin "6"
-		)
-		(pin "17"
-		)
-		(pin "14"
-		)
-		(pin "12"
-		)
-		(pin "4"
-		)
-		(pin "18"
-		)
-		(pin "5"
-		)
-		(pin "13"
-		)
-		(pin "15"
-		)
-		(pin "7"
-		)
-		(pin "30"
-		)
-		(pin "31"
-		)
-		(pin "2"
-		)
-		(pin "9"
-		)
-		(pin "8"
-		)
-		(pin "28"
-		)
-		(pin "23"
-		)
-		(pin "24"
-		)
-		(pin "27"
-		)
-		(pin "25"
-		)
-		(pin "26"
-		)
-		(pin "32"
-		)
-		(pin "1"
-		)
-		(pin "10"
-		)
-		(pin "29"
-		)
-		(pin "11"
-		)
-		(instances
-			(project ""
-				(path "/fcdc4d99-6273-4901-9910-bd8fd00b962f/aa87b2dd-90b3-41b3-8e99-8dcc5f11db59"
-					(reference "U201")
-					(unit 1)
-				)
