File: sensorpowerconversion.kicad_sch (KiCad schematic)
At the start: 13 parts

Commit message: Interactive BOM added. Updated Mega Symbol. Updated symbols in schematic. Generated production files.
Parts:
- R301: Manufacturer (none) -> UNI-ROYAL(Uniroyal Elec); Manufacturer Part No (none) -> 0805W8F2402T5E
- TP601: now left out of the parts list
Changed lines of the file:
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@@
 		(unit 1)
 		(exclude_from_sim no)
-		(in_bom yes)
+		(in_bom no)
 		(on_board yes)
 		(dnp no)
@@
 				(hide yes)
 			)
+		)
+		(property "Manufacturer" "UNI-ROYAL(Uniroyal Elec)"
+			(at 857.48 90.17 0)
+			(effects
+				(font
+					(size 1.27 1.27)
+				)
+				(justify left top)
+				(hide yes)
+			)
+		)
+		(property "Manufacturer Part No" "0805W8F2402T5E"
+			(at 957.48 90.17 0)
+			(effects
+				(font
+					(size 1.27 1.27)
+				)
+				(justify left top)
+				(hide yes)
+			)
