File: sensorrecievers.kicad_sch (KiCad schematic)
At the start: 40 parts, among them J304 1715747, U501 Precision ZD RR, U502 Precision ZD RR, U503 Precision ZD RR

Commit message: Removed one PTC per sensor as it shouldn't be required. Adjusted routing to star pattern.
Parts:
- removed F501, F504, F506: 50mA 30V, PTC, BOURNS Fuses:FUSC3226X110N, symbol BOURNS Fuses:MF-USMF005-2
Connections:
- net Sensor1: now also D502.2 (A2), D503.1 (A1), R501.1, R502.1
- net Sensor2: now also D505.2 (A2), D506.1 (A1), R506.1, R508.1
- net Sensor3: now also D508.2 (A2), D509.1 (A1), R511.1, R513.1

Commit message: Updated the diodes to fix issue. Now running 28V diodes for protection of sensing circuit.
Parts:
- removed D501, D502, D503, D504, D505, D506, D507, D508, D509: 13.3V 0.1uA Leak, LITTELFUSE Diodes:SODFL3619X98N, symbol LITTELFUSE Diodes:SMF4L13AT1G
- added D401, D402, D403, D404, D405, D406, D407, D408, D409: 28V 1uA Leak, LITTELFUSE Diodes:SODFL3619X98N, symbol LITTELFUSE Diodes:SMF28A
Connections:
- net GND: now also D401.2 (A2), D403.2 (A2), D404.2 (A2), D406.2 (A2), D407.2 (A2), D409.2 (A2)
- net Sensor1: now also D402.2 (A2), D403.1 (A1)
- net Sensor2: now also D405.2 (A2), D406.1 (A1)
- net Sensor3: now also D408.2 (A2), D409.1 (A1)
- net at F502.2, R501.2, R503.1: now also D401.1 (A1), D402.1 (A1)
- net at F505.2, R511.2, R512.1: now also D407.1 (A1), D408.1 (A1)
- net at F503.2, R506.2, R507.1: now also D404.1 (A1), D405.1 (A1)

Commit message: Interactive BOM added. Updated Mega Symbol. Updated symbols in schematic. Generated production files.
Parts:
- C501, C503, C505: Manufacturer (none) -> Samsung Electro-Mechanics; Manufacturer Part No (none) -> CL21B105KBFNNNE
- R502, R503, R504, R505, R507, R508, R509, R510, R512, R513, R514, R515: Manufacturer (none) -> UNI-ROYAL(Uniroyal Elec); Manufacturer Part No (none) -> 0805W8F1003T5E
