File: headers.kicad_sch (KiCad schematic)
At the start: 3 parts, among them J301 A2541WV-10P, J302 A2541WV-10P, J303 A2541WV-2x3P

Commit message: Redid the layout to shrink the board. Updated the silkscreen and updated the footprints to better reflect polarities and support a fab pdf.
Parts:
- J301, J302: now fitted; now in the parts list
Changed lines of the file:
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@@
 		(unit 1)
 		(exclude_from_sim no)
-		(in_bom no)
-		(on_board yes)
-		(dnp yes)
+		(in_bom yes)
+		(on_board yes)
+		(dnp no)
 		(fields_autoplaced yes)
 		(property "Reference" "J301"
@@
 		(unit 1)
 		(exclude_from_sim no)
-		(in_bom no)
-		(on_board yes)
-		(dnp yes)
+		(in_bom yes)
+		(on_board yes)
+		(dnp no)
 		(fields_autoplaced yes)
 		(property "Reference" "J302"

Commit message: Updated PCB, increased GND and improved connections on fills.
Parts:
- J303: footprint CJT Connectors:PinHeader_2x03_P2.54mm_Vertical -> CJT Connectors:PinHeader_2x03_P2.54mm_Vertical_Male
Changed lines of the file:
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@@
 			)
 		)
-		(property "Footprint" "CJT Connectors:PinHeader_2x03_P2.54mm_Vertical"
+		(property "Footprint" "CJT Connectors:PinHeader_2x03_P2.54mm_Vertical_Male"
 			(at 211.328 82.042 0)
 			(effects
